File: _autosave-STM32C071G8Ux.kicad_sch (KiCad schematic)
At the start: 38 parts, among them J1 UJ20-C-H-G-SMT-1-P16-TR, J2 Conn_01x14, J3 Conn_01x14, J4 Conn_ARM_SWD_TagConnect_TC203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, J5 Conn_ARM_JTAG_SWD_10, U1 STM32C071G8Ux, U2 USBLC6-2SC6, U4 TLV75533PDBV

Commit message: routing done but drc errors
Parts:
- renumbered C2 to C1, C1 to C2, C6 to C3, C3 to C4, C7 to C6, C4 to C7, D5 to D3, D6 to D4, D7 to D5, D8 to D6, D4 to D7, J3 to J1, J1 to J2, J2 to J3, JP4 to JP1, JP5 to JP2, JP2 to JP3, JP1 to JP4, JP3 to JP5, R5 to R2, R6 to R3, R2 to R4, R4 to R5, R7 to R6, U4 to U1, U1 to U3
Changed lines of the file:
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@@
 		(on_board yes)
 		(dnp no)
-		(property "Reference" "C2"
+		(property "Reference" "C1"
 			(at 25.146 97.028 0)
 			(effects
@@
 			(project "STM32C071G8Ux"
 				(path "/43830917-f7d7-4d02-b833-0362299cee99"
-					(reference "C2")
+					(reference "C1")
 					(unit 1)
 				)
@@
 		(dnp no)
 		(fields_autoplaced yes)
-		(property "Reference" "JP4"
+		(property "Reference" "JP1"
 			(at 257.81 153.67 0)
 			(effects
@@
 			(project "STM32C071G8Ux"
 				(path "/43830917-f7d7-4d02-b833-0362299cee99"
-					(reference "JP4")
+					(reference "JP1")
 					(unit 1)
 				)
@@
 		(dnp no)
 		(fields_autoplaced yes)
-		(property "Reference" "C4"
+		(property "Reference" "C7"
 			(at 198.12 53.3399 0)
 			(effects
@@
 			(project "STM32C071G8Ux"
 				(path "/43830917-f7d7-4d02-b833-0362299cee99"
-					(reference "C4")
+					(reference "C7")
 					(unit 1)
 				)
@@
 		(dnp no)
 		(fields_autoplaced yes)
-		(property "Reference" "U4"
+		(property "Reference" "U1"
 			(at 43.18 87.63 0)
 			(effects
@@
 			(project ""
 				(path "/43830917-f7d7-4d02-b833-0362299cee99"
-					(reference "U4")
+					(reference "U1")
 					(unit 1)
 				)
@@
 		(on_board yes)
 		(dnp no)
-		(property "Reference" "C6"
+		(property "Reference" "C3"
 			(at 17.526 97.028 0)
 			(effects
@@
 			(project "STM32C071G8Ux"
 				(path "/43830917-f7d7-4d02-b833-0362299cee99"
-					(reference "C6")
+					(reference "C3")
 					(unit 1)
 				)
@@
 		(dnp no)
 		(fields_autoplaced yes)
-		(property "Reference" "J1"
+		(property "Reference" "J2"
 			(at 34.29 17.78 0)
 			(effects
@@
 			(project ""
 				(path "/43830917-f7d7-4d02-b833-0362299cee99"
-					(reference "J1")
+					(reference "J2")
 					(unit 1)
 				)
@@
 		(on_board yes)
 		(dnp no)
-		(property "Reference" "U1"
+		(property "Reference" "U3"
 			(at 167.894 63.5 0)
 			(effects
@@
 			(project ""
 				(path "/43830917-f7d7-4d02-b833-0362299cee99"
-					(reference "U1")
+					(reference "U3")
 					(unit 1)
 				)
@@
 		(dnp no)
 		(fields_autoplaced yes)
-		(property "Reference" "J2"
+		(property "Reference" "J3"
 			(at 259.08 38.0999 0)
 			(effects
@@
 			(project ""
 				(path "/43830917-f7d7-4d02-b833-0362299cee99"
-					(reference "J2")
+					(reference "J3")
 					(unit 1)
 				)
@@
 		(dnp no)
 		(fields_autoplaced yes)
-		(property "Reference" "J3"
+		(property "Reference" "J1"
 			(at 259.08 91.4399 0)
 			(effects
@@
 			(project "STM32C071G8Ux"
 				(path "/43830917-f7d7-4d02-b833-0362299cee99"
-					(reference "J3")
+					(reference "J1")
 					(unit 1)
 				)
@@
 		(dnp no)
 		(fields_autoplaced yes)
-		(property "Reference" "JP2"
+		(property "Reference" "JP3"
 			(at 257.81 135.89 0)
 			(effects
@@
 			(project "STM32C071G8Ux"
 				(path "/43830917-f7d7-4d02-b833-0362299cee99"
-					(reference "JP2")
+					(reference "JP3")
 					(unit 1)
 				)
@@
 		(on_board yes)
 		(dnp no)
-		(property "Reference" "R4"
+		(property "Reference" "R5"
 			(at 105.41 72.136 90)
 			(effects
@@
 			(project "STM32C071G8Ux"
 				(path "/43830917-f7d7-4d02-b833-0362299cee99"
-					(reference "R4")
+					(reference "R5")
 					(unit 1)
 				)
@@
 		(on_board yes)
 		(dnp no)
-		(property "Reference" "D5"
+		(property "Reference" "D3"
 			(at 25.908 159.766 0)
 			(effects
@@
 			(project "STM32C071G8Ux"
 				(path "/43830917-f7d7-4d02-b833-0362299cee99"
-					(reference "D5")
+					(reference "D3")
 					(unit 1)
 				)
@@
 		(on_board yes)
 		(dnp no)
-		(property "Reference" "R7"
+		(property "Reference" "R6"
 			(at 93.472 32.766 0)
 			(effects
@@
 			(project "STM32C071G8Ux"
 				(path "/43830917-f7d7-4d02-b833-0362299cee99"
-					(reference "R7")
+					(reference "R6")
 					(unit 1)
 				)
@@
 		(dnp no)
 		(fields_autoplaced yes)
-		(property "Reference" "C7"
+		(property "Reference" "C6"
 			(at 114.3 124.4599 0)
 			(effects
@@
 			(project "STM32C071G8Ux"
 				(path "/43830917-f7d7-4d02-b833-0362299cee99"
-					(reference "C7")
+					(reference "C6")
 					(unit 1)
 				)
@@
 		(dnp no)
 		(fields_autoplaced yes)
-		(property "Reference" "JP3"
+		(property "Reference" "JP5"
 			(at 257.81 127 0)
 			(effects
@@
 			(project "STM32C071G8Ux"
 				(path "/43830917-f7d7-4d02-b833-0362299cee99"
-					(reference "JP3")
+					(reference "JP5")
 					(unit 1)
 				)
@@
 		(on_board yes)
 		(dnp no)
-		(property "Reference" "D8"
+		(property "Reference" "D6"
 			(at 25.908 178.816 0)
 			(effects
@@
 			(project "STM32C071G8Ux"
 				(path "/43830917-f7d7-4d02-b833-0362299cee99"
-					(reference "D8")
+					(reference "D6")
 					(unit 1)
 				)
@@
 		(on_board yes)
 		(dnp no)
-		(property "Reference" "R2"
+		(property "Reference" "R4"
 			(at 49.53 43.434 90)
 			(effects
@@
 			(project "STM32C071G8Ux"
 				(path "/43830917-f7d7-4d02-b833-0362299cee99"
-					(reference "R2")
+					(reference "R4")
 					(unit 1)
 				)
@@
 		(on_board yes)
 		(dnp no)
-		(property "Reference" "D6"
+		(property "Reference" "D4"
 			(at 25.908 166.116 0)
 			(effects
@@
 			(project "STM32C071G8Ux"
 				(path "/43830917-f7d7-4d02-b833-0362299cee99"
-					(reference "D6")
+					(reference "D4")
 					(unit 1)
 				)
@@
 		(on_board yes)
 		(dnp no)
-		(property "Reference" "D4"
+		(property "Reference" "D7"
 			(at 102.362 128.524 90)
 			(effects
@@
 			(project "STM32C071G8Ux"
 				(path "/43830917-f7d7-4d02-b833-0362299cee99"
-					(reference "D4")
+					(reference "D7")
 					(unit 1)
 				)
@@
 		(on_board yes)
 		(dnp no)
-		(property "Reference" "R6"
+		(property "Reference" "R3"
 			(at 105.41 87.376 90)
 			(effects
@@
 			(project "STM32C071G8Ux"
 				(path "/43830917-f7d7-4d02-b833-0362299cee99"
-					(reference "R6")
+					(reference "R3")
 					(unit 1)
 				)
@@
 		(dnp no)
 		(fields_autoplaced yes)
-		(property "Reference" "C1"
+		(property "Reference" "C2"
 			(at 60.96 97.7899 0)
 			(effects
@@
 			(project ""
 				(path "/43830917-f7d7-4d02-b833-0362299cee99"
-					(reference "C1")
+					(reference "C2")
 					(unit 1)
 				)
@@
 		(on_board yes)
 		(dnp no)
-		(property "Reference" "JP5"
+		(property "Reference" "JP2"
 			(at 257.81 119.888 0)
 			(effects
@@
 			(project "STM32C071G8Ux"
 				(path "/43830917-f7d7-4d02-b833-0362299cee99"
-					(reference "JP5")
+					(reference "JP2")
 					(unit 1)
 				)
@@
 		(on_board yes)
 		(dnp no)
-		(property "Reference" "D7"
+		(property "Reference" "D5"
 			(at 25.908 172.466 0)
 			(effects
@@
 			(project "STM32C071G8Ux"
 				(path "/43830917-f7d7-4d02-b833-0362299cee99"
-					(reference "D7")
+					(reference "D5")
 					(unit 1)
 				)
@@
 		(dnp no)
 		(fields_autoplaced yes)
-		(property "Reference" "C3"
+		(property "Reference" "C4"
 			(at 185.42 53.3399 0)
 			(effects
@@
 			(project "STM32C071G8Ux"
 				(path "/43830917-f7d7-4d02-b833-0362299cee99"
-					(reference "C3")
+					(reference "C4")
 					(unit 1)
 				)
@@
 		(dnp no)
 		(fields_autoplaced yes)
-		(property "Reference" "JP1"
+		(property "Reference" "JP4"
 			(at 257.81 144.78 0)
 			(effects
@@
 			(project ""
 				(path "/43830917-f7d7-4d02-b833-0362299cee99"
-					(reference "JP1")
+					(reference "JP4")
 					(unit 1)
 				)
@@
 		(on_board yes)
 		(dnp no)
-		(property "Reference" "R5"
+		(property "Reference" "R2"
 			(at 105.41 79.756 90)
 			(effects
@@
 			(project "STM32C071G8Ux"
 				(path "/43830917-f7d7-4d02-b833-0362299cee99"
-					(reference "R5")
+					(reference "R2")
 					(unit 1)
 				)
